File: hardware/board.brd (EAGLE design)
At the start: 53 x 30 mm, 45 parts, among them IC1 0915BM15A0001, J1 U.FL, U3 BLE113-A, X1 26MHz 10pF 10ppm -20C +70C, X3 MINI-USB-UX60-MB-5ST

Commit message: some edits made by jason
Parts:
- C2: device rcl:C0603K -> rcl:C0402K
- LED1: value red -> (none)
- LED2, LED5: value blue -> (none)
- LED3, LED4: value green -> (none)
- moved R3 1.20 mm to (20.7, 2.48)
- moved C9 0.96 mm to (25.1, 1.23), turned to 180 degrees
- moved C1 0.57 mm to (29.2, 7.04)
- moved LED2 0.51 mm to (51.6, 18.5)
- moved C7 0.38 mm to (22.3, 2.50)
- moved R12 0.27 mm to (49.9, 19.7), turned to 90 degrees
- moved R13 0.25 mm to (50.0, 23.0)
Routing:
- net DD: track 26.1 -> 30.2 mm
- net DD_BLE: track 28.7 -> 31.3 mm
- net MOSI: track 56.7 -> 58.5 mm
- net SCK: track 50.2 -> 51.8 mm
- net MISO: track 46.8 -> 48.3 mm
- net N$14: track 2.74 -> 4.23 mm
- net N$18: track 3.91 -> 5.30 mm
- net DC_BLE: track 19.8 -> 21.2 mm
- net VDD: track 152.6 -> 153.8 mm
- net DC: track 19.7 -> 20.6 mm
- net N$10: track 4.94 -> 5.85 mm
- net N$21: track 8.53 -> 9.30 mm
- net N$31: track 4.19 -> 3.41 mm
- net N$20: track 8.38 -> 9.15 mm
- net RESET: track 58.2 -> 58.9 mm
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