File: hardware/board.sch (EAGLE design)
At the start: 45 parts, among them IC1 0915BM15A0001, J1 U.FL, U3 BLE113-A, X1 26MHz 10pF 10ppm -20C +70C, X3 MINI-USB-UX60-MB-5ST

Commit message: some edits made by jason
Parts:
- C2: device rcl:C-USC0603K -> rcl:C-EUC0402K
- C3: device rcl:C-USC0603K -> rcl:C-EUC0603K
- LED1: value red -> (none)
- LED2, LED5: value blue -> (none)
- LED3, LED4: value green -> (none)
Changed lines of the file:
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@@
 <?xml version="1.0" encoding="utf-8"?>
 <!DOCTYPE eagle SYSTEM "eagle.dtd">
-<eagle version="7.1.0">
+<eagle version="7.2.0">
 <drawing>
 <settings>
@@
 <part name="JP1" library="SparkFun-Connectors" deviceset="M02" device="-JST-2MM-SMT"/>
 <part name="GND1" library="supply1" deviceset="GND" device=""/>
-<part name="C2" library="rcl" deviceset="C-US" device="C0603K" value="4.7uF"/>
+<part name="C2" library="rcl" deviceset="C-EU" device="C0402K" value="4.7uF"/>
 <part name="GND3" library="supply1" deviceset="GND" device=""/>
 <part name="R1" library="rcl" deviceset="R-US_" device="R0402" value="2K"/>
 <part name="R2" library="rcl" deviceset="R-US_" device="R0402" value="330"/>
-<part name="LED1" library="led" deviceset="LED" device="SML0603" value="red"/>
+<part name="LED1" library="led" deviceset="LED" device="SML0603"/>
 <part name="GND2" library="supply1" deviceset="GND" device=""/>
 <part name="GND4" library="supply1" deviceset="GND" device=""/>
-<part name="C3" library="rcl" deviceset="C-US" device="C0603K" value="4.7uF"/>
+<part name="C3" library="rcl" deviceset="C-EU" device="C0603K" value="4.7uF"/>
 <part name="GND5" library="supply1" deviceset="GND" device=""/>
 <part name="GND6" library="supply1" deviceset="GND" device=""/>
@@
 <part name="R11" library="rcl" deviceset="R-US_" device="R0402" value="470 ohms"/>
 <part name="SUPPLY10" library="supply2" deviceset="GND" device=""/>
-<part name="LED4" library="led" deviceset="LED" device="SML0603" value="green"/>
-<part name="LED5" library="led" deviceset="LED" device="SML0603" value="blue"/>
+<part name="LED4" library="led" deviceset="LED" device="SML0603"/>
+<part name="LED5" library="led" deviceset="LED" device="SML0603"/>
 <part name="SUPPLY11" library="supply2" deviceset="GND" device=""/>
 <part name="SUPPLY12" library="supply2" deviceset="GND" device=""/>
-<part name="LED2" library="led" deviceset="LED" device="SML0603" value="blue"/>
+<part name="LED2" library="led" deviceset="LED" device="SML0603"/>
 <part name="R12" library="rcl" deviceset="R-US_" device="R0402" value="470 ohms"/>
 <part name="SUPPLY13" library="supply2" deviceset="GND" device=""/>
-<part name="LED3" library="led" deviceset="LED" device="SML0603" value="green"/>
+<part name="LED3" library="led" deviceset="LED" device="SML0603"/>
 <part name="R13" library="rcl" deviceset="R-US_" device="R0402" value="470 ohms"/>
 <part name="C7" library="rcl" deviceset="C-EU" device="C0402" value="100nF"/>
